File: Sensor_Board_Rev1/tds.kicad_sch (KiCad schematic)
At the start: 36 parts, among them J4 XH2.54-2P, J5 Conn_01x03, U1 LMV324, U8 TPS60400DBVR, U9 XC6206P302MR

Commit message: Changing MPU6050 chip to MPU9250 breakout
Parts:
- U9: value XC6206P302MR -> XC6206P302MR-SOT23; VALUE XC6206P302MR-SOT23 -> (none)
